File: Production/SparkFun_Optical_Tracking_Odometry_Sensor-Panel.brd (EAGLE design)
At the start: 175 x 117.3 mm, 1830 parts, among them J1 QWIIC_RIGHT_ANGLE, J10 QWIIC_RIGHT_ANGLE, J11 QWIIC_RIGHT_ANGLE, J13 QWIIC_RIGHT_ANGLE, J14 QWIIC_RIGHT_ANGLE, J16 QWIIC_RIGHT_ANGLE, J17 QWIIC_RIGHT_ANGLE, J19 QWIIC_RIGHT_ANGLE, J2 QWIIC_RIGHT_ANGLE, J20 QWIIC_RIGHT_ANGLE, J22 QWIIC_RIGHT_ANGLE, J23 QWIIC_RIGHT_ANGLE, J25 QWIIC_RIGHT_ANGLE, J26 QWIIC_RIGHT_ANGLE, J28 QWIIC_RIGHT_ANGLE, J29 QWIIC_RIGHT_ANGLE, J31 QWIIC_RIGHT_ANGLE, J32 QWIIC_RIGHT_ANGLE, J34 QWIIC_RIGHT_ANGLE, J35 QWIIC_RIGHT_ANGLE, J37 QWIIC_RIGHT_ANGLE, J38 QWIIC_RIGHT_ANGLE, J4 QWIIC_RIGHT_ANGLE, J40 QWIIC_RIGHT_ANGLE, J41 QWIIC_RIGHT_ANGLE, J43 QWIIC_RIGHT_ANGLE, J44 QWIIC_RIGHT_ANGLE, J46 QWIIC_RIGHT_ANGLE, J47 QWIIC_RIGHT_ANGLE, J49 QWIIC_RIGHT_ANGLE, J5 QWIIC_RIGHT_ANGLE, J50 QWIIC_RIGHT_ANGLE, J52 QWIIC_RIGHT_ANGLE, J53 QWIIC_RIGHT_ANGLE, J55 QWIIC_RIGHT_ANGLE, J56 QWIIC_RIGHT_ANGLE, J58 QWIIC_RIGHT_ANGLE, J59 QWIIC_RIGHT_ANGLE, J61 QWIIC_RIGHT_ANGLE, J62 QWIIC_RIGHT_ANGLE, J64 QWIIC_RIGHT_ANGLE, J65 QWIIC_RIGHT_ANGLE, J67 QWIIC_RIGHT_ANGLE, J68 QWIIC_RIGHT_ANGLE, J7 QWIIC_RIGHT_ANGLE, J70 QWIIC_RIGHT_ANGLE, J71 QWIIC_RIGHT_ANGLE, J8 QWIIC_RIGHT_ANGLE, Q1 100mA/20V/3.8Ω, Q10 100mA/20V/3.8Ω, Q11 100mA/20V/3.8Ω, Q12 100mA/20V/3.8Ω, Q13 100mA/20V/3.8Ω, Q14 100mA/20V/3.8Ω, Q15 100mA/20V/3.8Ω, Q16 100mA/20V/3.8Ω, Q17 100mA/20V/3.8Ω, Q18 100mA/20V/3.8Ω, Q19 100mA/20V/3.8Ω, Q2 100mA/20V/3.8Ω, Q20 100mA/20V/3.8Ω, Q21 100mA/20V/3.8Ω, Q22 100mA/20V/3.8Ω, Q23 100mA/20V/3.8Ω, Q24 100mA/20V/3.8Ω, Q25 100mA/20V/3.8Ω, Q26 100mA/20V/3.8Ω, Q27 100mA/20V/3.8Ω, Q28 100mA/20V/3.8Ω, Q29 100mA/20V/3.8Ω, Q3 100mA/20V/3.8Ω, Q30 100mA/20V/3.8Ω, Q31 100mA/20V/3.8Ω, Q32 100mA/20V/3.8Ω, Q33 100mA/20V/3.8Ω, Q34 100mA/20V/3.8Ω, Q35 100mA/20V/3.8Ω, Q36 100mA/20V/3.8Ω, Q37 100mA/20V/3.8Ω, Q38 100mA/20V/3.8Ω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

Commit message: Add v11 production files
Parts:
- turned D1 to 180 degrees
- turned D13 to 180 degrees
- turned D17 to 180 degrees
- turned D21 to 180 degrees
- turned D25 to 180 degrees
- turned D29 to 180 degrees
- turned D33 to 180 degrees
- turned D37 to 180 degrees
- turned D41 to 180 degrees
- turned D45 to 180 degrees
- turned D49 to 180 degrees
- turned D5 to 180 degrees
- turned D53 to 180 degrees
- turned D57 to 180 degrees
- turned D61 to 180 degrees
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Connections:
- net GND: now also D1.C; no longer D1.A
- net GND1: now also D5.C; no longer D5.A
- net GND10: now also D41.C; no longer D41.A
- net GND11: now also D45.C; no longer D45.A
- net GND12: now also D49.C; no longer D49.A
- net GND13: now also D53.C; no longer D53.A
- net GND14: now also D57.C; no longer D57.A
- net GND15: now also D61.C; no longer D61.A
- net GND16: now also D65.C; no longer D65.A
- net GND17: now also D69.C; no longer D69.A
- net GND18: now also D73.C; no longer D73.A
- net GND19: now also D77.C; no longer D77.A
- net GND2: now also D9.C; no longer D9.A
- net GND20: now also D81.C; no longer D81.A
- net GND21: now also D85.C; no longer D85.A
- net GND22: now also D89.C; no longer D89.A
- net GND23: now also D93.C; no longer D93.A
- net GND3: now also D13.C; no longer D13.A
- net GND4: now also D17.C; no longer D17.A
- net GND5: now also D21.C; no longer D21.A
- net GND6: now also D25.C; no longer D25.A
- net GND7: now also D29.C; no longer D29.A
- net GND8: now also D33.C; no longer D33.A
- net GND9: now also D37.C; no longer D37.A
- net N$104: now also D49.A; no longer D49.C
- net N$112: now also D53.A; no longer D53.C
- net N$120: now also D57.A; no longer D57.C
- net N$128: now also D61.A; no longer D61.C
- net N$136: now also D65.A; no longer D65.C
- net N$144: now also D69.A; no longer D69.C
- net N$152: now also D73.A; no longer D73.C
- net N$16: now also D5.A; no longer D5.C
- net N$160: now also D77.A; no longer D77.C
- net N$168: now also D81.A; no longer D81.C
- net N$176: now also D85.A; no longer D85.C
- net N$184: now also D89.A; no longer D89.C
- net N$192: now also D93.A; no longer D93.C
- net N$2: now also D1.A; no longer D1.C
- net N$24: now also D9.A; no longer D9.C
- net N$32: now also D13.A; no longer D13.C
- net N$40: now also D17.A; no longer D17.C
- net N$48: now also D21.A; no longer D21.C
- net N$56: now also D25.A; no longer D25.C
- net N$64: now also D29.A; no longer D29.C
- net N$72: now also D33.A; no longer D33.C
- net N$80: now also D37.A; no longer D37.C
- net N$88: now also D41.A; no longer D41.C
- net N$96: now also D45.A; no longer D45.C
Other:
- board text added: "v11"
- board text removed: "v10"
